File: PCB/Starbie.kicad_pcb (KiCad board)
At the start: 2 copper layers, 110 x 110 mm, 8 parts, among them J1 Conn_01x04_Pin, J2 Conn_01x08_Pin, SW1 SW_Push, SW2 SW_Push, U1 XIAO-ESP32-C3-SMD, U2 DHT11

Commit message: Add files via upload
Parts:
- moved U1 21.4 mm to (121.4, 102.0), turned to 90 degrees
Routing:
- net +3.3V: track 269.3 -> 161.7 mm
- net /DHT11 Data: track 102.6 -> 192.3 mm, vias 0 -> 2
- net /GPIO3: track 141.9 -> 74.8 mm
- net /SDA: track 126.4 -> 96.4 mm, vias 1 -> 0
- net /SCL: track 118.3 -> 100.0 mm, vias 1 -> 0
- net /GPIO2: track 38.8 -> 49.9 mm
- net GND: track 239.1 -> 243.1 mm, vias 0 -> 1

Commit message: Add files via upload
Parts:
- moved U1 7.91 mm to (116.9, 108.5)
- moved SW2 6.23 mm to (177.5, 122.9)
- moved SW1 6.20 mm to (136.5, 122.4)
- moved U2 4.92 mm to (152.9, 65.5)
Routing:
- net /DHT11 Data: track 192.3 -> 148.4 mm
- net /SDA: track 96.4 -> 121.2 mm
- net GND: track 243.1 -> 267.3 mm, vias 1 -> 0
- net /GPIO2: track 49.9 -> 38.7 mm
- net +3.3V: track 161.7 -> 172.4 mm, vias 0 -> 2
- net /GPIO3: track 74.8 -> 80.3 mm
- net /SCL: track 100.0 -> 97.0 mm
